Commit message: Add support for Gen 3 Lite grippers

File: pykin/assets/urdf/gen3_lite/6dof/GEN3-LITE.urdf (robot description, URDF)
Before this commit: robot KR7108-URDF, 8 links, 7 joints
Links:
- removed link DUMMY
- removed link END_EFFECTOR
- added link GRIPPER_FRAME, mass 0.1395; collision mesh filename=meshes/gripper_base_link.STL; visual mesh filename=meshes/gripper_base_link.STL
- added link LEFT_FINGER_DIST, mass 0.010748; collision mesh filename=meshes/left_finger_dist_link.STL; visual mesh filename=meshes/left_finger_dist_link.STL
- added link LEFT_FINGER_PROX, mass 0.018385; collision mesh filename=meshes/left_finger_prox_link.STL; visual mesh filename=meshes/left_finger_prox_link.STL
- added link RIGHT_FINGER_DIST, mass 0.010748; collision mesh filename=meshes/right_finger_dist_link.STL; visual mesh filename=meshes/right_finger_dist_link.STL
- added link RIGHT_FINGER_PROX, mass 0.018385; collision mesh filename=meshes/right_finger_prox_link.STL; visual mesh filename=meshes/right_finger_prox_link.STL
Joints:
- removed joint END_EFFECTOR
- added joint LEFT_BOTTOM: type revolute, parent GRIPPER_FRAME, child LEFT_FINGER_PROX, origin xyz=0 0.0305 0.070003 rpy=0 1.5708 0, axis 0 0 1, limit lower=-0.96 upper=0.09 effort=1000 velocity=1000
- added joint LEFT_TIP: type revolute, parent LEFT_FINGER_PROX, child LEFT_FINGER_DIST, origin xyz=-0.045636 -0.020423 6.9901E-05 rpy=0 0 0, axis 0 0 -1, limit lower=-0.21 upper=1.03 effort=1000 velocity=1000
- added joint RIGHT_BOTTOM: type revolute, parent GRIPPER_FRAME, child RIGHT_FINGER_PROX, origin xyz=0 -0.030501 0.070003 rpy=0 1.5708 0, axis 0 0 1, limit lower=-0.09 upper=0.96 effort=1000 velocity=1000
- added joint RIGHT_TIP: type revolute, parent RIGHT_FINGER_PROX, child RIGHT_FINGER_DIST, origin xyz=-0.045636 0.020423 0 rpy=0 0 0, axis 0 0 1, limit lower=-1.03 upper=0.21 effort=1000 velocity=1000
- joint J5: child END_EFFECTOR -> GRIPPER_FRAME
